File: reverse_polarity_protection.kicad_sch (KiCad schematic)
At the start: 3 parts, among them Q1 Q_Toshiba_SSM3J328R

Commit message: sch: first draft
Parts:
- Q1: value Q_Toshiba_SSM3J328R -> Q_Toshiba_SSM3J351R
Changed lines of the file:
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@@
 			)
 		)
-		(property "Value" "Q_Toshiba_SSM3J328R"
+		(property "Value" "Q_Toshiba_SSM3J351R"
 			(at 50.8 22.86 90)
 			(effects
