File: project-hw-60v-dcdc.kicad_sch (KiCad schematic)
At the start: 0 parts

Commit message: sch: first draft
Parts:
- added J1, J2, J3, J4: Conn_01x01_Socket, Connector_SolderPad:EdgePad_1x1, symbol Connector:Conn_01x01_Socket
Connections:
- net Reverse Polarity Protection/IN: now also J1.1 (Pin_1)
- new net GND: J2.1 (Pin_1), J4.1 (Pin_1)
- new net LMR516x5 Converter/Vout: J3.1 (Pin_1)
Other:
- sheet LMR516x5 Converter ports: added Vout; removed 5V

Commit message: First placement
Parts:
- J1, J2, J3: footprint Connector_SolderPad:EdgePad_1x1 -> Connector_SolderPad:EdgePad_1x1_Short
Connections:
- net Reverse Polarity Protection/IN is gone; now on net LMR516x5 Converter/Vin: J1.1 (Pin_1)
Other:
- removed sheet Reverse Polarity Protection
- moved on the sheet: J3, J4

Commit message: First routing
Parts:
- removed J4: Conn_01x01_Socket, Connector_SolderPad:EdgePad_1x1, symbol Connector:Conn_01x01_Socket
Changed lines of the file:
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@@
 	(wire
 		(pts
-			(xy 73.66 33.02) (xy 76.2 33.02)
+			(xy 30.48 27.94) (xy 38.1 27.94)
 		)
 		(stroke
@@
 	(wire
 		(pts
-			(xy 30.48 27.94) (xy 38.1 27.94)
+			(xy 33.02 35.56) (xy 33.02 38.1)
 		)
 		(stroke
@@
 	(wire
 		(pts
-			(xy 33.02 35.56) (xy 33.02 38.1)
+			(xy 30.48 26.67) (xy 30.48 27.94)
 		)
 		(stroke
@@
 		)
 	)
-	(wire
-		(pts
-			(xy 30.48 26.67) (xy 30.48 27.94)
-		)
-		(stroke
-			(width 0)
-			(type default)
-		)
-	)
-	(wire
-		(pts
-			(xy 73.66 33.02) (xy 73.66 38.1)
-		)
-		(stroke
-			(width 0)
-			(type default)
-		)
-	)
 	(symbol
 		(lib_id "Connector:Conn_01x01_Socket")
@@
 	(symbol
 		(lib_id "power:GND")
-		(at 73.66 38.1 0)
-		(unit 1)
-		(exclude_from_sim no)
-		(in_bom yes)
-		(on_board yes)
-		(dnp no)
-		(fields_autoplaced yes)
-		(property "Reference" "#PWR03"
-			(at 73.66 44.45 0)
-			(effects
-				(font
-					(size 1.27 1.27)
-				)
-				(hide yes)
-			)
-		)
-		(property "Value" "GND"
-			(at 73.66 43.18 0)
-			(effects
-				(font
-					(size 1.27 1.27)
-				)
-			)
-		)
-		(property "Footprint" ""
-			(at 73.66 38.1 0)
-			(effects
-				(font
-					(size 1.27 1.27)
-				)
-				(hide yes)
-			)
-		)
-		(property "Datasheet" ""
-			(at 73.66 38.1 0)
-			(effects
-				(font
-					(size 1.27 1.27)
-				)
-				(hide yes)
-			)
-		)
-		(property "Description" "Power symbol creates a global label with name \"GND\" , ground"
-			(at 73.66 38.1 0)
-			(effects
-				(font
-					(size 1.27 1.27)
-				)
-				(hide yes)
-			)
-		)
-		(pin "1"
-		)
-		(instances
-			(project "project-hw-60v-dcdc"
-				(path "/bf513276-35b6-4c64-961b-f9ab0be6dcba"
-					(reference "#PWR03")
-					(unit 1)
-				)
-			)
-		)
-	)
-	(symbol
-		(lib_id "power:GND")
 		(at 33.02 38.1 0)
 		(unit 1)
@@
 					(unit 1)
 				)
-			)
-		)
-	)
-	(symbol
-		(lib_id "Connector:Conn_01x01_Socket")
-		(at 81.28 33.02 0)
-		(unit 1)
-		(exclude_from_sim no)
-		(in_bom yes)
-		(on_board yes)
-		(dnp no)
-		(fields_autoplaced yes)
-		(property "Reference" "J4"
-			(at 82.55 33.0199 0)
-			(effects
-				(font
-					(size 1.27 1.27)
-				)
-				(justify left)
-			)
-		)
-		(property "Value" "Conn_01x01_Socket"
-			(at 80.645 35.56 0)
-			(effects
-				(font
-					(size 1.27 1.27)
-				)
-				(hide yes)
-			)
-		)
-		(property "Footprint" "Connector_SolderPad:EdgePad_1x1"
-			(at 81.28 33.02 0)
-			(effects
-				(font
-					(size 1.27 1.27)
-				)
-				(hide yes)
-			)
-		)
-		(property "Datasheet" "~"
-			(at 81.28 33.02 0)
-			(effects
-				(font
-					(size 1.27 1.27)
-				)
-				(hide yes)
-			)
-		)
-		(property "Description" "Generic connector, single row, 01x01, script generated"
-			(at 81.28 33.02 0)
-			(effects
-				(font
-					(size 1.27 1.27)
-				)
-				(hide yes)
-			)
-		)
-		(pin "1"
-		)
-		(instances
-			(project "project-hw-60v-dcdc"
-				(path "/bf513276-35b6-4c64-961b-f9ab0be6dcba"
-					(reference "J4")
-					(unit 1)
-				)
