File: project-hw-60v-dcdc.kicad_pcb (KiCad board)
At the start: 2 copper layers, 26 x 20 mm, 17 parts, among them J1 Conn_01x01_Socket, J2 Conn_01x01_Socket, J3 Conn_01x01_Socket, J4 Conn_01x01_Socket, Q1 Q_Toshiba_SSM3J351R, U1 LMR516x5

Commit message: Add assembly file
Parts:
- C3: value 0.1uF -> 1uF 100V
Changed lines of the file:
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@@
 		)
 		(property "Value" "10uF 50V"
-			(at 0 2.3 90)
+			(at 3 -2.25 180)
 			(layer "F.Fab")
 			(effects
@@
 		)
 		(property "Value" "0.1uF"
-			(at 0 1.43 90)
+			(at 0 1 90)
 			(layer "F.Fab")
 			(effects
@@
 		)
 		(property "Value" "10uF 100V"
-			(at 0 2.3 90)
+			(at 3 2.75 180)
 			(layer "F.Fab")
 			(effects
@@
 		)
 		(property "Value" "LMR516x5"
-			(at 0 3 0)
+			(at 0.5 5.5 90)
 			(layer "F.Fab")
 			(effects
@@
 		)
 		(property "Value" "10uF 50V"
-			(at 0 2.3 90)
-			(layer "F.Fab")
+			(at -1 -2.5 90)
+			(layer "F.Fab")
+			(hide yes)
 			(effects
 				(font
@@
 			(unlocked yes)
 			(layer "F.Fab")
+			(hide yes)
 			(effects
 				(font
@@
 			(unlocked yes)
 			(layer "F.Fab")
+			(hide yes)
 			(effects
 				(font
@@
 			(unlocked yes)
 			(layer "F.Fab")
+			(hide yes)
 			(effects
 				(font
@@
 			(unlocked yes)
 			(layer "F.Fab")
+			(hide yes)
 			(effects
 				(font
@@
 			(unlocked yes)
 			(layer "F.Fab")
+			(hide yes)
 			(effects
 				(font
@@
 			(unlocked yes)
 			(layer "F.Fab")
+			(hide yes)
 			(effects
 				(font
@@
 		)
 		(property "Value" "MM5Z5V1T5GF"
-			(at 0 2 90)
+			(at -2 -4.75 180)
 			(layer "F.Fab")
 			(effects
@@
 			(at 0 -2 90)
 			(layer "F.Fab")
+			(hide yes)
 			(effects
 				(font
@@
 		)
 		(property "Value" "6.8uH"
-			(at 0 4 0)
+			(at 3.75 -2.25 90)
 			(unlocked yes)
 			(layer "F.Fab")
@@
 		)
 		(property "Value" "Q_Toshiba_SSM3J351R"
-			(at 0 3 0)
+			(at 2.25 -6 90)
 			(layer "F.Fab")
 			(effects
@@
 		)
 		(property "Value" "100k"
-			(at 0 1.43 0)
+			(at 1.25 -1.25 0)
 			(layer "F.Fab")
 			(effects
@@
 			)
 		)
-		(property "Value" "0.1uF"
-			(at 0 1.43 90)
+		(property "Value" "1uF 100V"
+			(at 5 0 90)
 			(layer "F.Fab")
 			(effects
@@
 			)
 		)
-		(property "Description" "Unpolarized capacitor, small symbol"
+		(property "Description" "C1608X7R2A105K080AC"
 			(at 0 0 -90)
 			(unlocked yes)
@@
 			(unlocked yes)
 			(layer "F.Fab")
+			(hide yes)
 			(effects
 				(font
@@
 			(unlocked yes)
 			(layer "F.Fab")
+			(hide yes)
 			(effects
 				(font
@@
 		)
 		(property "Value" "10uF 100V"
-			(at 0 2.3 90)
-			(layer "F.Fab")
+			(at 0 3.25 90)
+			(layer "F.Fab")
+			(hide yes)
 			(effects
 				(font
@@
 		)
 		(property "Value" "Vchoice"
-			(at 0 1.43 90)
-			(layer "F.Fab")
-			(effects
+			(at 1 1.25 90)
+			(layer "F.Fab")
+			(effects

Commit message: First placement
Parts:
- removed D1: MM5Z5V1T5GF, SOT:D_SOD-523
- removed Q1: Q_Toshiba_SSM3J351R, SOT:SOT-23F
- removed R1: 100k, Resistor_SMD:R_0603_1608Metric
- added C7: Csnub, Capacitor_SMD:C_0402_1005Metric, F.Cu at (71.9, 31.8)
- added R4: Rsnub, Resistor_SMD:R_0402_1005Metric, F.Cu at (71.9, 32.7)
- C1, C2: footprint Capacitor_SMD:C_1210_3225Metric -> SMD:C_1210_3225Metric_Tight
- C3, C4: footprint Capacitor_SMD:C_0603_1608Metric -> SMD:C_0603_1608Metric_Tight
- J1, J2, J3: footprint Connector_SolderPad:EdgePad_1x1 -> Connector_SolderPad:EdgePad_1x1_Short
- R2: footprint SMD:0603_1608Metric_DNI_NoPaste -> Resistor_SMD:R_0603_1608Metric
- U1: footprint SOT:TSOT-23-6 -> SOT:TSOT-23-6_Tight
- moved J2 32.5 mm to (74.5, 37.8)
- moved C2 29.3 mm to (68.8, 37.5), turned to 0 degrees
- moved J1 29.2 mm to (65.2, 31.5), turned to 0 degrees
- moved C1 25.4 mm to (68.8, 34.7), turned to 0 degrees
- moved J3 25.3 mm to (79.2, 27.0), turned to 180 degrees
- moved C5 22.9 mm to (74.9, 33.6)
- moved C3 22.8 mm to (69.3, 32.7), turned to 0 degrees
- moved C6 22.6 mm to (78.1, 33.6)
- moved U1 21.1 mm to (69.0, 30.5)
- moved C4 21.0 mm to (70.4, 27.8)
- moved R2 20.8 mm to (65.8, 27.0)
- moved R3 20.8 mm to (67.2, 27.0)
- moved L1 20.3 mm to (74.2, 28.0)
- moved J4 19.1 mm to (37.0, 50.8)
Connections:
- net Net-(U1-FB) renamed /LMR516x5 Converter/FB
- J1 pad 1: /Reverse Polarity Protection/IN -> /LMR516x5 Converter/Vin
Routing:
- net /LMR516x5 Converter/Vout: track 12.6 -> 0.00 mm, vias 2 -> 0
- net Net-(D1-A): track 4.08 -> 0.00 mm
- net Net-(U1-CB): track 1.86 -> 0.00 mm
- net GND: vias 22 -> 0
- removed copper zone on F.Cu, net /Reverse Polarity Protection/IN
Other:
- board size 26 x 20 mm -> 57 x 20 mm
- copper layers 2 -> 4

Commit message: First routing
Parts:
- removed J4: Conn_01x01_Socket, Connector_SolderPad:EdgePad_1x1
- moved J3 29.7 mm to (49.8, 30.0)
- moved C4 29.6 mm to (40.9, 30.3)
- moved C1 29.6 mm to (39.3, 37.2)
- moved C2 29.6 mm to (39.3, 40.0)
- moved C3 29.6 mm to (39.8, 35.2)
- moved J1 29.6 mm to (35.8, 34.0)
- moved J2 29.6 mm to (45.0, 40.2)
- moved U1 29.6 mm to (39.5, 33.0)
- moved L1 29.5 mm to (44.8, 30.4)
- moved C7 29.5 mm to (42.6, 35.2), turned to 180 degrees
- moved R4 29.3 mm to (42.6, 34.2), turned to 0 degrees
- moved C5 29.3 mm to (45.7, 36.1)
- moved C6 29.3 mm to (48.9, 36.1)
- moved R2 29.3 mm to (36.6, 29.7)
- moved R3 29.3 mm to (38.1, 29.7)
Connections:
- C7 pad 1: Net-(U1-SW) -> Net-(C7-Pad1)
- C7 pad 2: Net-(C7-Pad2) -> GND
- R4 pad 1: Net-(C7-Pad2) -> Net-(U1-SW)
- R4 pad 2: GND -> Net-(C7-Pad1)
Routing:
- net /LMR516x5 Converter/Vout: track 0.00 -> 24.5 mm, vias 0 -> 2
- net Net-(U1-CB): track 0.00 -> 1.02 mm
- net Net-(C7-Pad1): track 0.00 -> 1.01 mm
- net GND: vias 0 -> 19
Other:
- board size 57 x 20 mm -> 17.5 x 15 mm
- board text removed: "GND"
- board text removed: "V_{IN}"
- board text removed: "V_{OUT}"

Commit message: Add inner ground planes
Routing:
- added copper zone on In1.Cu, net GND
- added copper zone on In2.Cu, net GND
Changed lines of the file:
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@@
+		(net 1)
+		(net_name "GND")
+		(layers "In1.Cu" "In2.Cu")
+		(hatch edge 0.5)
+		(priority 1)
+		(connect_pads
+			(clearance 0.25)
+		)
+		(min_thickness 0.25)
+		(filled_areas_thickness no)
+		(fill yes
+			(thermal_gap 0.5)
+			(thermal_bridge_width 0.5)
+			(smoothing fillet)
+			(radius 0.5)
+		)
+		(polygon
+			(pts
+				(xy 34 27) (xy 34 42) (xy 51.5 42) (xy 51.5 27)
+			)
+		)
+	)
+	(zone
 		(net 1)
 		(net_name "GND")
