File: project-hw-60v-dcdc.kicad_pcb (KiCad board)
At the start: 4 copper layers, 17.5 x 15 mm, 15 parts, among them J1 Conn_01x01_Socket, J2 Conn_01x01_Socket, J3 Conn_01x01_Socket, U1 LMR516x5

Commit message: Add copper pour under the inductor
Routing:
- net GND: vias 22 -> 26
Changed lines of the file:
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@@
 			(net 3 "Net-(U1-SW)")
 			(pintype "passive")
+			(clearance 0.4)
 		)
 		(model "${KIPRJMOD}/kicad-library/3dmodels/C_0603_1608Metric.step"
@@
 			(pinfunction "1")
 			(pintype "passive")
+			(clearance 0.4)
 		)
 		(pad "2" smd roundrect
@@
 	)
 	(via
+		(at 44.8 30.2)
+		(size 0.6)
+		(drill 0.3)
+		(layers "F.Cu" "B.Cu")
+		(free yes)
+		(net 1)
+	)
+	(via
 		(at 41.7 36.9)
 		(size 0.6)
@@
 	)
 	(via
+		(at 44.8 28)
+		(size 0.6)
+		(drill 0.3)
+		(layers "F.Cu" "B.Cu")
+		(free yes)
+		(net 1)
+	)
+	(via
 		(at 41.7 36.3)
 		(size 0.6)
@@
 	)
 	(via
+		(at 44.8 32.2)
+		(size 0.6)
+		(drill 0.3)
+		(layers "F.Cu" "B.Cu")
+		(free yes)
+		(net 1)
+	)
+	(via
 		(at 46.6 38.5)
 		(size 0.6)
@@
 	)
 	(via
+		(at 44.8 31.2)
+		(size 0.6)
+		(drill 0.3)
+		(layers "F.Cu" "B.Cu")
+		(free yes)
+		(net 1)
+	)
+	(via
 		(at 41.7 40.3)
 		(size 0.6)
@@
 			)
 		)
-	)
-	(zone
-		(net 0)
-		(net_name "")
-		(layer "F.Cu")
-		(hatch edge 0.5)
-		(connect_pads yes
-			(clearance 0)
-		)
-		(min_thickness 0.25)
-		(filled_areas_thickness no)
-		(keepout
-			(tracks allowed)
-			(vias allowed)
-			(pads allowed)
-			(copperpour not_allowed)
-			(footprints allowed)
-		)
-		(fill
-			(thermal_gap 0.25)
-			(thermal_bridge_width 0.5)
-		)
-		(polygon
-			(pts
-				(xy 40.3 27) (xy 40.3 29) (xy 43.7 29) (xy 43.7 33.8) (xy 44.8 33.8) (xy 44.8 27)
-			)
-		)

Commit message: Change ground silkscreen
Other:
- board text added: "GND"
Changed lines of the file:
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@@
-	)
-	(gr_line
-		(start 47.45 40.6)
-		(end 48.45 40.6)
-		(stroke
-			(width 0.2)
-			(type default)
-		)
-		(layer "F.SilkS")
-	)
-	(gr_line
-		(start 47.95 41.2)
-		(end 48.45 40.6)
-		(stroke
-			(width 0.2)
-			(type default)
-		)
-		(layer "F.SilkS")
 	)
 	(gr_line
@@
 	)
 	(gr_line
-		(start 47.95 40.6)
-		(end 47.95 39.8)
-		(stroke
-			(width 0.2)
-			(type default)
-		)
-		(layer "F.SilkS")
-	)
-	(gr_line
 		(start 50.3 33.3)
 		(end 50.8 32.8)
@@
 		(start 35.85 37.35)
 		(end 36.35 36.85)
-		(stroke
-			(width 0.2)
-			(type default)
-		)
-		(layer "F.SilkS")
-	)
-	(gr_line
-		(start 47.45 40.6)
-		(end 47.95 41.2)
 		(stroke
 			(width 0.2)
@@
 				)
 			)
+		)
+	)
+	(gr_text "GND"
+		(at 47.2 41.4 0)
+		(layer "F.SilkS")
+		(effects
+			(font
+				(face "FreeSans")
+				(size 1.1 1.1)
+				(thickness 0.24)
+				(bold yes)
+			)
+			(justify left bottom)
+		)
+		(render_cache "GND" 0
+			(polygon
+				(pts
+					(xy 48.079078 40.439238) (xy 48.056206 40.384749) (xy 48.026211 40.339495) (xy 47.980813 40.297382)
+					(xy 47.925158 40.268567) (xy 47.870943 40.254714) (xy 47.809605 40.250096) (xy 47.748305 40.25529)
+					(xy 47.692996 40.270872) (xy 47.643678 40.296841) (xy 47.600351 40.333199) (xy 47.578283 40.358638)
+					(xy 47.545412 40.410072) (xy 47.523662 40.460441) (xy 47.507844 40.516609) (xy 47.497958 40.578576)
+					(xy 47.494251 40.634646) (xy 47.493921 40.658202) (xy 47.497104 40.721599) (xy 47.506654 40.780613)
+					(xy 47.522569 40.835245) (xy 47.544851 40.885494) (xy 47.573498 40.931361) (xy 47.584462 40.945676)
+					(xy 47.626478 40.989539) (xy 47.673302 41.022629) (xy 47.724934 41.044945) (xy 47.781374 41.056488)
+					(xy 47.815785 41.058247) (xy 47.866025 41.052874) (xy 47.917994 41.037335) (xy 47.935073 41.030575)
+					(xy 47.982929 41.005534) (xy 48.009225 40.986782) (xy 48.046997 40.946981) (xy 48.069675 40.911018)
+					(xy 48.090967 40.859031) (xy 48.101778 40.804193) (xy 48.102184 40.800327) (xy 47.845338 40.800327)
+					(xy 47.845338 40.611185) (xy 48.297236 40.611185) (xy 48.297236 41.213) (xy 48.157798 41.213) (xy 48.129856 41.074099)
+					(xy 48.092181 41.12103) (xy 48.051999 41.160268) (xy 48.00441 41.194843) (xy 47.984508 41.206014)
+					(xy 47.930968 41.227833) (xy 47.877085 41.24056) (xy 47.817804 41.246742) (xy 47.789724 41.247389)
+					(xy 47.733677 41.244799) (xy 47.680124 41.237028) (xy 47.61669 41.220031) (xy 47.557152 41.194939)
+					(xy 47.501509 41.161753) (xy 47.449763 41.120473) (xy 47.411172 41.081621) (xy 47.376161 41.03879)
+					(xy 47.345819 40.993179) (xy 47.320144 40.94479) (xy 47.299138 40.893621) (xy 47.282799 40.839674)
+					(xy 47.271129 40.782947) (xy 47.264127 40.723442) (xy 47.261793 40.661157) (xy 47.264161 40.595963)
+					(xy 47.271263 40.53391) (xy 47.283102 40.474996) (xy 47.299675 40.419222) (xy 47.320984 40.366589)
+					(xy 47.347028 40.317095) (xy 47.377807 40.270742) (xy 47.413321 40.227528) (xy 47.452698 40.188488)
+					(xy 47.494929 40.154653) (xy 47.551732 40.119679) (xy 47.612995 40.092838) (xy 47.665218 40.077222)
+					(xy 47.720294 40.066811) (xy 47.778226 40.061606) (xy 47.808262 40.060955) (xy 47.870293 40.063447)
+					(xy 47.928769 40.070925) (xy 47.983689 40.083387) (xy 48.035055 40.100835) (xy 48.092001 40.128353)
+					(xy 48.143827 40.163048) (xy 48.189332 40.203783) (xy 48.22711 40.249618) (xy 48.257162 40.300553)
+					(xy 48.279487 40.356589) (xy 48.294087 40.417726) (xy 48.297236 40.439238)
+				)
+			)
+			(polygon
+				(pts
+					(xy 49.19351 41.213) (xy 48.740268 40.428491) (xy 48.740268 41.213) (xy 48.50814 41.213) (xy 48.50814 40.07815)
+					(xy 48.746448 40.07815) (xy 49.19351 40.850299) (xy 49.19351 40.07815) (xy 49.425638 40.07815)
+					(xy 49.425638 41.213)
+				)
+			)
+			(polygon
+				(pts
+					(xy 50.163459 40.079641) (xy 50.220538 40.084997) (xy 50.277968 40.09568) (xy 50.322986 40.109315)
+					(xy 50.373062 40.13244) (xy 50.417838 40.162859) (xy 50.457315 40.200573) (xy 50.464574 40.20899)
+					(xy 50.50428 40.263125) (xy 50.531199 40.310155) (xy 50.553811 40.360492) (xy 50.572116 40.414137)
+					(xy 50.586114 40.47109) (xy 50.595805 40.531352) (xy 50.601189 40.594921) (xy 50.6024 40.644769)
+					(xy 50.600247 40.711524) (xy 50.593786 40.77477) (xy 50.583018 40.834506) (xy 50.567943 40.890733)
+					(xy 50.548562 40.943451) (xy 50.524873 40.992659) (xy 50.489205 41.049234) (xy 50.464574 41.080547)
+					(xy 50.418588 41.12556) (xy 50.372964 41.155957) (xy 50.320703 41.179886) (xy 50.261803 41.197348)
+					(xy 50.196266 41.208343) (xy 50.139056 41.212482) (xy 50.108859 41.213) (xy 49.667707 41.213) (xy 49.667707 41.023858)
+					(xy 49.899836 41.023858) (xy 50.108859 41.023858) (xy 50.170127 41.01796) (xy 50.223227 41.000266)
+					(xy 50.268157 40.970775) (xy 50.304918 40.929489) (xy 50.33351 40.876406) (xy 50.353933 40.811527)
+					(xy 50.36389 40.755126) (xy 50.369251 40.692091) (xy 50.370272 40.646381) (xy 50.367974 40.578633)
+					(xy 50.361081 40.517549) (xy 50.349593 40.463129) (xy 50.327128 40.400935) (xy 50.296494 40.350587)
+					(xy 50.25769 40.312086) (xy 50.210718 40.285431) (xy 50.155576 40.270623) (xy 50.108859 40.267291)
+					(xy 49.899836 40.267291) (xy 49.899836 41.023858) (xy 49.667707 41.023858) (xy 49.667707 40.07815)
+					(xy 50.108859 40.07815)
+				)
+			)
